File: Lars-10W-RGBW-V1/Driver.kicad_sch (KiCad schematic)
At the start: 12 parts, among them U202 TPS92201

Commit message: Fixed via sizes
Parts:
- R201: footprint Resistor_SMD:R_0402_1005Metric -> Resistor_SMD:R_0805_2012Metric
Changed lines of the file:
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@@
 			)
 		)
-		(property "Footprint" "Resistor_SMD:R_0402_1005Metric"
+		(property "Footprint" "Resistor_SMD:R_0805_2012Metric"
 			(at 153.67 79.248 90)
 			(effects
